File: feather-decagon.sch (KiCad schematic (older format))
At the start: 19 parts

Commit message: update
Parts:
- removed U? (x4): GND, symbol Adafruit-FONA-800-GSM-Breakout-eagle-import:GND
- gave numbers to parts that had none: 15
Connections:
- net labels added: GND
Changed lines of the file:
@@
 $Descr User 11984 8268
 encoding utf-8
-Sheet 1 1
+Sheet 1 2
 Title ""
 Date ""
@@
 $EndDescr
 $Comp
-L quahog_0.1:q_data_header U?
+L quahog_0.1:q_data_header U4
 U 1 1 5CC25294
 P 6300 2700
-F 0 "U?" H 6480 2952 50  0000 L CNN
+F 0 "U4" H 6480 2952 50  0000 L CNN
 F 1 "q_data_header" H 6480 2859 50  0000 L CNN
 F 2 "" H 6300 2700 50  0001 C CNN
@@
 $EndComp
 $Comp
-L Connector:VX7805 U?
+L Connector:VX7805 U1
 U 1 1 5CC255DA
 P 2350 1400
-F 0 "U?" H 2631 1447 50  0000 L CNN
+F 0 "U1" H 2631 1447 50  0000 L CNN
 F 1 "VX7803" H 2631 1354 50  0000 L CNN
 F 2 "" H 2350 1400 50  0001 C CNN
@@
 $EndComp
 $Comp
-L tpl5110:tpl5110 U?
+L tpl5110:tpl5110 U2
 U 1 1 5CC34CA2
 P 2850 2550
-F 0 "U?" H 2825 3071 50  0000 C CNN
+F 0 "U2" H 2825 3071 50  0000 C CNN
 F 1 "tpl5110" H 2825 2978 50  0000 C CNN
 F 2 "" H 3250 2450 50  0001 C CNN
@@
 $EndComp
 $Comp
-L device:Q_NPN_EBC Q?
+L device:Q_NPN_EBC Q1
 U 1 1 5CC34FFB
 P 3550 5250
-F 0 "Q?" H 3741 5297 50  0000 L CNN
+F 0 "Q1" H 3741 5297 50  0000 L CNN
 F 1 "Q_NPN_EBC" H 3741 5204 50  0000 L CNN
 F 2 "TO_SOT_Packages_THT:TO-92_Molded_Wide" H 3750 5350 50  0001 C CNN
@@
 $EndComp
 $Comp
-L device:Q_PMOS_GDS Q?
+L device:Q_PMOS_GDS Q3
 U 1 1 5CC35002
 P 3650 4700
-F 0 "Q?" V 3996 4700 50  0000 C CNN
+F 0 "Q3" V 3996 4700 50  0000 C CNN
 F 1 "Q_PMOS_GDS" V 3903 4700 50  0000 C CNN
 F 2 "TO_SOT_Packages_THT:TO-220-3_Vertical" H 3850 4800 50  0001 C CNN
@@
 $EndComp
 $Comp
-L device:R R?
+L device:R R2
 U 1 1 5CC35009
 P 3200 5250
-F 0 "R?" V 2990 5250 50  0000 C CNN
+F 0 "R2" V 2990 5250 50  0000 C CNN
 F 1 "10K" V 3083 5250 50  0000 C CNN
 F 2 "Resistors_THT:R_Axial_DIN0414_L11.9mm_D4.5mm_P15.24mm_Horizontal" V 3130 5250 50  0001 C CNN
@@
 $EndComp
 $Comp
-L device:R R?
+L device:R R1
 U 1 1 5CC35010
 P 3200 4750
-F 0 "R?" H 3130 4703 50  0000 R CNN
+F 0 "R1" H 3130 4703 50  0000 R CNN
 F 1 "100K" H 3130 4796 50  0000 R CNN
 F 2 "Resistors_THT:R_Axial_DIN0414_L11.9mm_D4.5mm_P15.24mm_Horizontal" V 3130 4750 50  0001 C CNN
@@
 	3200 4600 3450 4600
 $Comp
-L Connector:Screw_Terminal_01x02 J?
+L Connector:Screw_Terminal_01x02 J1
 U 1 1 5CC36E5B
 P 1250 750
-F 0 "J?" V 1215 559 50  0000 R CNN
+F 0 "J1" V 1215 559 50  0000 R CNN
 F 1 "Screw_Terminal_01x02" V 1122 559 50  0000 R CNN
 F 2 "" H 1250 750 50  0001 C CNN
@@
 	2200 2300 2250 2300
 $Comp
-L Connector:Conn_01x02 J?
+L Connector:Conn_01x02 J2
 U 1 1 5CC49BA2
 P 2250 3250
-F 0 "J?" V 2121 3330 50  0000 L CNN
+F 0 "J2" V 2121 3330 50  0000 L CNN
 F 1 "Conn_01x02" V 2214 3330 50  0000 L CNN
 F 2 "" H 2250 3250 50  0001 C CNN
@@
 	3400 2600 4100 2600
 $Comp
-L Connector:Conn_01x16 J?
+L Connector:Conn_01x16 J3
 U 1 1 5CC58770
 P 4650 2550
-F 0 "J?" H 4568 1519 50  0000 C CNN
+F 0 "J3" H 4568 1519 50  0000 C CNN
 F 1 "Conn_01x16" H 4568 1612 50  0000 C CNN
 F 2 "" H 4650 2550 50  0001 C CNN
@@
 	4850 3050 5200 3050
 $Comp
-L Adafruit-FONA-800-GSM-Breakout-eagle-import:GND U?
+L Adafruit-FONA-800-GSM-Breakout-eagle-import:GND #U0101
 U 1 1 5CC8E15B
 P 4400 4050
-F 0 "U?" H 4450 4100 50  0001 C CNN
+F 0 "#U0101" H 4450 4100 50  0001 C CNN
 F 1 "GND" H 4481 4086 42  0000 L CNN
 F 2 "" H 4400 4050 50  0001 C CNN
@@
 	2150 2450 2150 3050
 $Comp
-L Adafruit-FONA-800-GSM-Breakout-eagle-import:GND U?
+L Adafruit-FONA-800-GSM-Breakout-eagle-import:GND #U0102
 U 1 1 5CCB358B
 P 1900 2550
-F 0 "U?" H 1950 2600 50  0001 C CNN
+F 0 "#U0102" H 1950 2600 50  0001 C CNN
 F 1 "GND" H 1981 2586 42  0000 L CNN
 F 2 "" H 1900 2550 50  0001 C CNN
@@
 	1550 1300 2200 1300
 $Comp
-L Adafruit-FONA-800-GSM-Breakout-eagle-import:GND U?
+L Adafruit-FONA-800-GSM-Breakout-eagle-import:GND #U0103
 U 1 1 5CCC87ED
 P 3650 5750
-F 0 "U?" H 3700 5800 50  0001 C CNN
+F 0 "#U0103" H 3700 5800 50  0001 C CNN
 F 1 "GND" H 3731 5786 42  0000 L CNN
 F 2 "" H 3650 5750 50  0001 C CNN
@@
 Connection ~ 5200 3050
 $Comp
-L device:Q_NPN_EBC Q?
+L device:Q_NPN_EBC Q2
 U 1 1 5CCFA3CF
 P 3550 7100
-F 0 "Q?" H 3741 7147 50  0000 L CNN
+F 0 "Q2" H 3741 7147 50  0000 L CNN
 F 1 "Q_NPN_EBC" H 3741 7054 50  0000 L CNN
 F 2 "TO_SOT_Packages_THT:TO-92_Molded_Wide" H 3750 7200 50  0001 C CNN
@@
 $EndComp
 $Comp
-L device:Q_PMOS_GDS Q?
+L device:Q_PMOS_GDS Q4
 U 1 1 5CCFA3D6
 P 3650 6550
-F 0 "Q?" V 3996 6550 50  0000 C CNN
+F 0 "Q4" V 3996 6550 50  0000 C CNN
 F 1 "Q_PMOS_GDS" V 3903 6550 50  0000 C CNN
 F 2 "TO_SOT_Packages_THT:TO-220-3_Vertical" H 3850 6650 50  0001 C CNN
@@
 $EndComp
 $Comp
-L device:R R?
+L device:R R4
 U 1 1 5CCFA3DD
 P 3200 7100
-F 0 "R?" V 2990 7100 50  0000 C CNN
+F 0 "R4" V 2990 7100 50  0000 C CNN
 F 1 "10K" V 3083 7100 50  0000 C CNN
 F 2 "Resistors_THT:R_Axial_DIN0414_L11.9mm_D4.5mm_P15.24mm_Horizontal" V 3130 7100 50  0001 C CNN
@@
 $EndComp
 $Comp
-L device:R R?
+L device:R R3
 U 1 1 5CCFA3E4
 P 3200 6600
-F 0 "R?" H 3130 6553 50  0000 R CNN
+F 0 "R3" H 3130 6553 50  0000 R CNN
 F 1 "100K" H 3130 6646 50  0000 R CNN
 F 2 "Resistors_THT:R_Axial_DIN0414_L11.9mm_D4.5mm_P15.24mm_Horizontal" V 3130 6600 50  0001 C CNN
@@
 	2450 7100 3050 7100
 $Comp
-L Adafruit-FONA-800-GSM-Breakout-eagle-import:GND U?
+L Adafruit-FONA-800-GSM-Breakout-eagle-import:GND #U0104
 U 1 1 5CCFA3F3
 P 3650 7600
-F 0 "U?" H 3700 7650 50  0001 C CNN
+F 0 "#U0104" H 3700 7650 50  0001 C CNN
 F 1 "GND" H 3731 7636 42  0000 L CNN
 F 2 "" H 3650 7600 50  0001 C CNN
@@
 	5000 3250 6100 3250
 $Comp
-L quahog_0.1:adafruit_bme280 U?
+L quahog_0.1:adafruit_bme280 U3
 U 1 1 5CD68BDB
 P 6200 4200
-F 0 "U?" H 6481 4402 50  0000 L CNN
+F 0 "U3" H 6481 4402 50  0000 L CNN
 F 1 "adafruit_bme280" H 6481 4309 50  0000 L CNN
 F 2 "" H 6200 4200 50  0001 C CNN
@@
 	4900 3950 4400 3950
 Connection ~ 4900 3950
+$Sheet
+S 8050 1650 1250 1300
+U 5CC38A02
+F0 "Sheet5CC38A01" 50
+F1 "file5CC38A01.sch" 50
+$EndSheet
 $EndSCHEMATC
